File: CAN_LIGHT/_autosave-CAN_LIGHT.kicad_sch (KiCad schematic)
At the start: 1 part, among them U1 TCAN334

Commit message: Place caps
Parts:
- added C1, C10, C11, C12, C13, C14, C15, C16, C17, C18, C19, C2, C20, C21, C22, C23, C24, C25, C26, C27, C28, C29, C3, C30, C31, C32, C33, C34, C35, C36, C37, C38, C39, C4, C40, C41, C42, C44, C5, C6, C7, C8, C9: 0.1uF, Capacitor_SMD:C_0603_1608Metric_Pad1.08x0.95mm_HandSolder, symbol Device:C
- added C43: 10uF, Capacitor_SMD:C_0603_1608Metric_Pad1.08x0.95mm_HandSolder, symbol Device:C
- added C45: 10nF, Capacitor_SMD:C_0603_1608Metric_Pad1.08x0.95mm_HandSolder, symbol Device:C
- added D1, D10, D11, D12, D13, D14, D15, D16, D17, D18, D19, D2, D20, D21, D22, D23, D24, D25, D26, D27, D28, D29, D3, D30, D31, D32, D33, D34, D35, D36, D37, D38, D39, D4, D40, D41, D42, D5, D6, D7, D8, D9: ~, IN-PI4818QAS5R5G5BPW:INPI4818QAS5R5G5BPW, symbol LED:IN-PI4818QAS5R5G5BPW
- added IC1: MSPM0C1103SDDFR, SOT65P280X110-8N, symbol MSPM0C1103SDDFR:MSPM0C1103SDDFR
- added J1: Conn_ARM_SWD_TagConnect_TC2030, Connector:Tag-Connect_TC2030-IDC-FP_2x03_P1.27mm_Vertical, symbol Connector:Conn_ARM_SWD_TagConnect_TC2030
- added J2: 436500401, 436500401:MOLEX_436500401, symbol 0436500401:436500401
- added JP1: SolderJumper_2_Open, symbol Jumper:SolderJumper_2_Open
- added R1: 47K, Resistor_SMD:R_0603_1608Metric_Pad0.98x0.95mm_HandSolder, symbol Device:R_US
- added R2: 2.2K, Resistor_SMD:R_0603_1608Metric_Pad0.98x0.95mm_HandSolder, symbol Device:R_US
- added R3: 500, Resistor_SMD:R_0603_1608Metric_Pad0.98x0.95mm_HandSolder, symbol Device:R_US
- added R4: 169K, Resistor_SMD:R_0603_1608Metric_Pad0.98x0.95mm_HandSolder, symbol Device:R_US
- added R5: 301K, Resistor_SMD:R_0603_1608Metric_Pad0.98x0.95mm_HandSolder, symbol Device:R_US
- added U2: TPS76333DBVR, DBV5, symbol TPS76333DBVR:TPS76333DBVR
- added U3: NCV891330PD50R2G, SOIC8_3P9X4P9_ONS, symbol NCV891330PD50R2G:NCV891330PD50R2G
Connections:
- net at U1.1 (TXD): now also IC1.8 (PA24_/_A3/UART_RX)
- net GND: now reaches U1.2 (GND)
- net GND: now also C1.2, C10.2, C11.2, C12.2, C13.2, C14.2, C15.2, C16.2, C17.2, C18.2, C19.2, C2.2, C20.2, C21.2, C22.2, C23.2, C24.2, C25.2, C26.2, C27.2, C28.2, C29.2, C3.2, C30.2, C31.2, C32.2, C33.2, C34.2, C35.2, C36.2, C37.2, C38.2, C39.2, C4.2, C40.2, C41.2, C42.2, C43.2, C44.2, C45.2, C5.2, C6.2, C7.2, C8.2, C9.2, D1.4 (GND), D10.4 (GND), D11.4 (GND), D12.4 (GND), D13.4 (GND), D14.4 (GND), D15.4 (GND), D16.4 (GND), D17.4 (GND), D18.4 (GND), D19.4 (GND), D2.4 (GND), D20.4 (GND), D21.4 (GND), D22.4 (GND), D23.4 (GND), D24.4 (GND), D25.4 (GND), D26.4 (GND), D27.4 (GND), D28.4 (GND), D29.4 (GND), D3.4 (GND), D30.4 (GND), D31.4 (GND), D32.4 (GND), D33.4 (GND), D34.4 (GND), D35.4 (GND), D36.4 (GND), D37.4 (GND), D38.4 (GND), D39.4 (GND), D4.4 (GND), D40.4 (GND), D41.4 (GND), D42.4 (GND), D5.4 (GND), D6.4 (GND), D7.4 (GND), D8.4 (GND), D9.4 (GND), IC1.3 (VSS), J1.5 (GND), J2.2, R4.2, U2.2 (GND), U3.4 (GND)
- net +3.3V: now reaches U1.3 (VCC)
- net +3.3V: now also C43.1, C44.1, IC1.4 (VDD), R1.1, R5.2, U2.5 (OUT)
- net at U1.4 (RXD): now also IC1.1 (PA27_/_A0/UART_TX)
- net at U1.6 (CANL): now also J2.4
- net at U1.7 (CANH): now also J2.3
- new net: D11.3 (DOUT), D12.6 (DIN)
- new net: D10.3 (DOUT), D11.6 (DIN)
- new net: D5.3 (DOUT), D6.6 (DIN)
- new net: D4.3 (DOUT), D5.6 (DIN)
- new net: D35.3 (DOUT), D36.6 (DIN)
- new net: D34.3 (DOUT), D35.6 (DIN)
- new net: D1.3 (DOUT), D2.6 (DIN)
- new net: D1.6 (DIN), R3.2
- new net: R4.1, R5.1, U2.4 (NC/FB)
- new net: D14.3 (DOUT), D15.6 (DIN)
- new net: D13.3 (DOUT), D14.6 (DIN)
- new net: C45.1, IC1.2 (PA1_/_NRST), J1.3 (~{RESET}), R1.2
- new net: IC1.5 (PA0), R2.2, R3.1
- new net: IC1.6 (PA19_/_SWDIO), J1.2 (SWDIO)
- new net: IC1.7 (PA20_/_A6_/_SWCLK), J1.4 (SWCLK)
- new net: D12.3 (DOUT), D13.6 (DIN)
- new net: D3.3 (DOUT), D4.6 (DIN)
- new net: D36.3 (DOUT), D37.6 (DIN)
- new net: D24.3 (DOUT), D25.6 (DIN)
- new net: D23.3 (DOUT), D24.6 (DIN)
- new net: D33.3 (DOUT), D34.6 (DIN)
- new net: D37.3 (DOUT), D38.6 (DIN)
- new net: D32.3 (DOUT), D33.6 (DIN)
- new net: JP1.1 (A), U2.3 (EN)
- new net: D15.3 (DOUT), D16.6 (DIN)
- new net: D31.3 (DOUT), D32.6 (DIN)
- new net: D30.3 (DOUT), D31.6 (DIN)
- new net: D6.3 (DOUT), D7.6 (DIN)
- new net: D41.3 (DOUT), D42.6 (DIN)
- new net: D17.3 (DOUT), D18.6 (DIN)
- new net: D16.3 (DOUT), D17.6 (DIN)
- new net: D39.3 (DOUT), D40.6 (DIN)
- new net: D38.3 (DOUT), D39.6 (DIN)
- new net: D25.3 (DOUT), D26.6 (DIN)
- new net: D7.3 (DOUT), D8.6 (DIN)
- new net: D40.3 (DOUT), D41.6 (DIN)
- new net: D21.3 (DOUT), D22.6 (DIN)
- new net: D20.3 (DOUT), D21.6 (DIN)
- new net: D2.3 (DOUT), D3.6 (DIN)
- new net: D22.3 (DOUT), D23.6 (DIN)
- new net: D27.3 (DOUT), D28.6 (DIN)
- new net: D26.3 (DOUT), D27.6 (DIN)
- new net: D19.3 (DOUT), D20.6 (DIN)
- new net: D18.3 (DOUT), D19.6 (DIN)
- new net: D10.6 (DIN), D9.3 (DOUT)
- new net: D8.3 (DOUT), D9.6 (DIN)
- new net: D29.3 (DOUT), D30.6 (DIN)
- new net: D28.3 (DOUT), D29.6 (DIN)
- new net +12V: J2.1, U3.1 (VIN), U3.5 (EN)
- new net +5V: C1.1, C10.1, C11.1, C12.1, C13.1, C14.1, C15.1, C16.1, C17.1, C18.1, C19.1, C2.1, C20.1, C21.1, C22.1, C23.1, C24.1, C25.1, C26.1, C27.1, C28.1, C29.1, C3.1, C30.1, C31.1, C32.1, C33.1, C34.1, C35.1, C36.1, C37.1, C38.1, C39.1, C4.1, C40.1, C41.1, C42.1, C5.1, C6.1, C7.1, C8.1, C9.1, D1.1 (W-VDD), D1.5 (VDD), D10.1 (W-VDD), D10.5 (VDD), D11.1 (W-VDD), D11.5 (VDD), D12.1 (W-VDD), D12.5 (VDD), D13.1 (W-VDD), D13.5 (VDD), D14.1 (W-VDD), D14.5 (VDD), D15.1 (W-VDD), D15.5 (VDD), D16.1 (W-VDD), D16.5 (VDD), D17.1 (W-VDD), D17.5 (VDD), D18.1 (W-VDD), D18.5 (VDD), D19.1 (W-VDD), D19.5 (VDD), D2.1 (W-VDD), D2.5 (VDD), D20.1 (W-VDD), D20.5 (VDD), D21.1 (W-VDD), D21.5 (VDD), D22.1 (W-VDD), D22.5 (VDD), D23.1 (W-VDD), D23.5 (VDD), D24.1 (W-VDD), D24.5 (VDD), D25.1 (W-VDD), D25.5 (VDD), D26.1 (W-VDD), D26.5 (VDD), D27.1 (W-VDD), D27.5 (VDD), D28.1 (W-VDD), D28.5 (VDD), D29.1 (W-VDD), D29.5 (VDD), D3.1 (W-VDD), D3.5 (VDD), D30.1 (W-VDD), D30.5 (VDD), D31.1 (W-VDD), D31.5 (VDD), D32.1 (W-VDD), D32.5 (VDD), D33.1 (W-VDD), D33.5 (VDD), D34.1 (W-VDD), D34.5 (VDD), D35.1 (W-VDD), D35.5 (VDD), D36.1 (W-VDD), D36.5 (VDD), D37.1 (W-VDD), D37.5 (VDD), D38.1 (W-VDD), D38.5 (VDD), D39.1 (W-VDD), D39.5 (VDD), D4.1 (W-VDD), D4.5 (VDD), D40.1 (W-VDD), D40.5 (VDD), D41.1 (W-VDD), D41.5 (VDD), D42.1 (W-VDD), D42.5 (VDD), D5.1 (W-VDD), D5.5 (VDD), D6.1 (W-VDD), D6.5 (VDD), D7.1 (W-VDD), D7.5 (VDD), D8.1 (W-VDD), D8.5 (VDD), D9.1 (W-VDD), D9.5 (VDD), JP1.2 (B), R2.1, U2.1 (IN), U3.6 (VOUT)
- no-connect marks 0 -> 1
Other:
- moved on the sheet: U1

Commit message: Export initial STEP file to print
Parts:
- removed J2: 436500401, 436500401:MOLEX_436500401, symbol 0436500401:436500401
- added C46, C47, C48, C49, C50, C51, C52, C53, C54, C55, C56, C57, C58, C59, C60, C61, C62, C63, C64, C65, C66, C67, C68, C69, C70, C71, C72, C73, C74, C75, C76, C77, C78, C79, C80, C81, C82, C83, C84, C85, C86, C87: 0.1uF, Capacitor_SMD:C_0603_1608Metric_Pad1.08x0.95mm_HandSolder, symbol Device:C
- added D43, D44, D45, D46, D47, D48, D49, D50, D51, D52, D53, D54, D55, D56, D57, D58, D59, D60, D61, D62, D63, D64, D65, D66, D67, D68, D69, D70, D71, D72, D73, D74, D75, D76, D77, D78, D79, D80, D81, D82, D83, D84: ~, IN-PI4818QAS5R5G5BPW:INPI4818QAS5R5G5BPW, symbol LED:IN-PI4818QAS5R5G5BPW
- added J2: 436500428, 436500428:CON_436500428_MOL, symbol 436500428:436500428
- added J3: 430450428, 430450428:CON_430450428_MOL, symbol 430450428:430450428
- renumbered IC1 to U1, U1 to U2, U2 to U3, U3 to U4
Connections:
- net +12V: now also J2.1
- net +5V: now also C46.1, C47.1, C48.1, C49.1, C50.1, C51.1, C52.1, C53.1, C54.1, C55.1, C56.1, C57.1, C58.1, C59.1, C60.1, C61.1, C62.1, C63.1, C64.1, C65.1, C66.1, C67.1, C68.1, C69.1, C70.1, C71.1, C72.1, C73.1, C74.1, C75.1, C76.1, C77.1, C78.1, C79.1, C80.1, C81.1, C82.1, C83.1, C84.1, C85.1, C86.1, C87.1, D43.1 (W-VDD), D43.5 (VDD), D44.1 (W-VDD), D44.5 (VDD), D45.1 (W-VDD), D45.5 (VDD), D46.1 (W-VDD), D46.5 (VDD), D47.1 (W-VDD), D47.5 (VDD), D48.1 (W-VDD), D48.5 (VDD), D49.1 (W-VDD), D49.5 (VDD), D50.1 (W-VDD), D50.5 (VDD), D51.1 (W-VDD), D51.5 (VDD), D52.1 (W-VDD), D52.5 (VDD), D53.1 (W-VDD), D53.5 (VDD), D54.1 (W-VDD), D54.5 (VDD), D55.1 (W-VDD), D55.5 (VDD), D56.1 (W-VDD), D56.5 (VDD), D57.1 (W-VDD), D57.5 (VDD), D58.1 (W-VDD), D58.5 (VDD), D59.1 (W-VDD), D59.5 (VDD), D60.1 (W-VDD), D60.5 (VDD), D61.1 (W-VDD), D61.5 (VDD), D62.1 (W-VDD), D62.5 (VDD), D63.1 (W-VDD), D63.5 (VDD), D64.1 (W-VDD), D64.5 (VDD), D65.1 (W-VDD), D65.5 (VDD), D66.1 (W-VDD), D66.5 (VDD), D67.1 (W-VDD), D67.5 (VDD), D68.1 (W-VDD), D68.5 (VDD), D69.1 (W-VDD), D69.5 (VDD), D70.1 (W-VDD), D70.5 (VDD), D71.1 (W-VDD), D71.5 (VDD), D72.1 (W-VDD), D72.5 (VDD), D73.1 (W-VDD), D73.5 (VDD), D74.1 (W-VDD), D74.5 (VDD), D75.1 (W-VDD), D75.5 (VDD), D76.1 (W-VDD), D76.5 (VDD), D77.1 (W-VDD), D77.5 (VDD), D78.1 (W-VDD), D78.5 (VDD), D79.1 (W-VDD), D79.5 (VDD), D80.1 (W-VDD), D80.5 (VDD), D81.1 (W-VDD), D81.5 (VDD), D82.1 (W-VDD), D82.5 (VDD), D83.1 (W-VDD), D83.5 (VDD), D84.1 (W-VDD), D84.5 (VDD)
- net GND: now also C46.2, C47.2, C48.2, C49.2, C50.2, C51.2, C52.2, C53.2, C54.2, C55.2, C56.2, C57.2, C58.2, C59.2, C60.2, C61.2, C62.2, C63.2, C64.2, C65.2, C66.2, C67.2, C68.2, C69.2, C70.2, C71.2, C72.2, C73.2, C74.2, C75.2, C76.2, C77.2, C78.2, C79.2, C80.2, C81.2, C82.2, C83.2, C84.2, C85.2, C86.2, C87.2, D43.4 (GND), D44.4 (GND), D45.4 (GND), D46.4 (GND), D47.4 (GND), D48.4 (GND), D49.4 (GND), D50.4 (GND), D51.4 (GND), D52.4 (GND), D53.4 (GND), D54.4 (GND), D55.4 (GND), D56.4 (GND), D57.4 (GND), D58.4 (GND), D59.4 (GND), D60.4 (GND), D61.4 (GND), D62.4 (GND), D63.4 (GND), D64.4 (GND), D65.4 (GND), D66.4 (GND), D67.4 (GND), D68.4 (GND), D69.4 (GND), D70.4 (GND), D71.4 (GND), D72.4 (GND), D73.4 (GND), D74.4 (GND), D75.4 (GND), D76.4 (GND), D77.4 (GND), D78.4 (GND), D79.4 (GND), D80.4 (GND), D81.4 (GND), D82.4 (GND), D83.4 (GND), D84.4 (GND), J2.2
- net at D42.3 (DOUT): now also D43.6 (DIN)
- net at U2.7 (CANH): now also J2.3
- net at U2.6 (CANL): now also J2.4
- new net: D81.3 (DOUT), D82.6 (DIN)
- new net: D80.3 (DOUT), D81.6 (DIN)
- new net: D69.3 (DOUT), D70.6 (DIN)
- new net: D68.3 (DOUT), D69.6 (DIN)
- new net: D67.3 (DOUT), D68.6 (DIN)
- new net: D61.3 (DOUT), D62.6 (DIN)
- new net: D60.3 (DOUT), D61.6 (DIN)
- new net: D71.3 (DOUT), D72.6 (DIN)
- new net: D70.3 (DOUT), D71.6 (DIN)
- new net: D47.3 (DOUT), D48.6 (DIN)
- new net: D46.3 (DOUT), D47.6 (DIN)
- new net: D74.3 (DOUT), D75.6 (DIN)
- new net: D73.3 (DOUT), D74.6 (DIN)
- new net: D59.3 (DOUT), D60.6 (DIN)
- new net: D54.3 (DOUT), D55.6 (DIN)
- new net: D53.3 (DOUT), D54.6 (DIN)
- new net: D43.3 (DOUT), D44.6 (DIN)
- new net: D77.3 (DOUT), D78.6 (DIN)
- new net: D76.3 (DOUT), D77.6 (DIN)
- new net: D83.3 (DOUT), D84.6 (DIN)
- new net: D82.3 (DOUT), D83.6 (DIN)
- new net: D65.3 (DOUT), D66.6 (DIN)
- new net: D64.3 (DOUT), D65.6 (DIN)
- new net: D72.3 (DOUT), D73.6 (DIN)
- new net: D44.3 (DOUT), D45.6 (DIN)
- new net: D62.3 (DOUT), D63.6 (DIN)
- new net: D63.3 (DOUT), D64.6 (DIN)
- new net: D75.3 (DOUT), D76.6 (DIN)
- new net: D56.3 (DOUT), D57.6 (DIN)
- new net: D55.3 (DOUT), D56.6 (DIN)
- new net: D48.3 (DOUT), D49.6 (DIN)
- new net: D78.3 (DOUT), D79.6 (DIN)
- new net: D49.3 (DOUT), D50.6 (DIN)
- new net: D58.3 (DOUT), D59.6 (DIN)
- new net: D57.3 (DOUT), D58.6 (DIN)
- new net: D79.3 (DOUT), D80.6 (DIN)
- new net: D52.3 (DOUT), D53.6 (DIN)
- new net: D51.3 (DOUT), D52.6 (DIN)
- new net: D45.3 (DOUT), D46.6 (DIN)
- new net: D66.3 (DOUT), D67.6 (DIN)
- new net: D50.3 (DOUT), D51.6 (DIN)
Other:
- moved on the sheet: C1, C10, C11, C12, C13, C14, C15, C16, C17, C18, C19, C2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
